File: UccMicroDuino/UccMicroDuino.kicad_pcb (KiCad board)
At the start: 2 copper layers, 8 parts, among them J1 Conn_01x10_Socket, J2 USB_A, U1 ATtiny85-20S

Commit message: Placa prueba didactica
Parts:
- added D4: LED, ledSmd:ledSMD, F.Cu at (191.8, 77.0)
- added D5: D_Zener, Diode_SMD:D_SOD-123, F.Cu at (209.1, 65.6)
- added R2: R, Resistor_SMD:R_0805_2012Metric_Pad1.20x1.40mm_HandSolder, F.Cu at (187.0, 77.0)
- added R3: R, Resistor_SMD:R_0805_2012Metric_Pad1.20x1.40mm_HandSolder, F.Cu at (187.8, 84.0)
- added R4: R, Resistor_SMD:R_0805_2012Metric_Pad1.20x1.40mm_HandSolder, F.Cu at (202.4, 65.4)
- added R5: R, Resistor_SMD:R_0805_2012Metric_Pad1.20x1.40mm_HandSolder, F.Cu at (212.0, 65.0)
- moved J1 104.7 mm to (225.4, 94.4), turned to -90 degrees
- moved U1 82.7 mm to (214.3, 85.4)
- moved D2 79.6 mm to (205.0, 66.0), turned to -90 degrees
- moved D1 73.9 mm to (199.0, 61.8), turned to 90 degrees
- moved J2 73.3 mm to (203.0, 54.0), turned to -90 degrees
- moved R1 60.5 mm to (199.0, 66.8), turned to -90 degrees
- moved D3 57.1 mm to (192.8, 84.0)
- moved C1 44.4 mm to (182.8, 71.0)
Connections:
- C1 pad 1: unconnected-(C1-Pad1) -> +5V
- C1 pad 2: unconnected-(C1-Pad2) -> GND
- D1 pad 2: unconnected-(D1-A-Pad2) -> Net-(D1-A)
- D2 pad 1: unconnected-(D2-K-Pad1) -> Net-(D2-K)
- D2 pad 2: unconnected-(D2-A-Pad2) -> GND
- D3 pad 1: unconnected-(D3-K-Pad1) -> Net-(D3-K)
- D3 pad 2: unconnected-(D3-A-Pad2) -> +5V
- J1 pad 1: unconnected-(J1-Pin_1-Pad1) -> +5V
- J1 pad 10: unconnected-(J1-Pin_10-Pad10) -> Net-(J1-Pin_10)
- J1 pad 2: unconnected-(J1-Pin_2-Pad2) -> GND
- J1 pad 4: unconnected-(J1-Pin_4-Pad4) -> Net-(J1-Pin_4)
- J1 pad 5: unconnected-(J1-Pin_5-Pad5) -> Net-(D4-A)
- J1 pad 6: unconnected-(J1-Pin_6-Pad6) -> Net-(J1-Pin_6)
- J1 pad 7: unconnected-(J1-Pin_7-Pad7) -> Net-(J1-Pin_7)
- J1 pad 8: unconnected-(J1-Pin_8-Pad8) -> Net-(J1-Pin_8)
- J2 pad 1: unconnected-(J2-VBUS-Pad1) -> Net-(D1-A)
- J2 pad 2: unconnected-(J2-D--Pad2) -> Net-(D2-K)
- J2 pad 3: unconnected-(J2-D+-Pad3) -> Net-(D5-K)
- R1 pad 2: unconnected-(R1-Pad2) -> Net-(D5-K)
- U1 pad 1: unconnected-(U1-~{RESET}/PB5-Pad1) -> Net-(J1-Pin_10)
- U1 pad 2: unconnected-(U1-XTAL1/PB3-Pad2) -> Net-(J1-Pin_7)
- U1 pad 3: unconnected-(U1-XTAL2/PB4-Pad3) -> Net-(J1-Pin_8)
- U1 pad 4: unconnected-(U1-GND-Pad4) -> GND
- U1 pad 5: unconnected-(U1-AREF/PB0-Pad5) -> Net-(J1-Pin_4)
- U1 pad 6: unconnected-(U1-PB1-Pad6) -> Net-(D4-A)
- U1 pad 7: unconnected-(U1-PB2-Pad7) -> Net-(J1-Pin_6)
- U1 pad 8: unconnected-(U1-VCC-Pad8) -> +5V
Routing:
- net Net-(D1-A): track 0.00 -> 0.71 mm
- net Net-(D2-K): track 0.00 -> 0.67 mm
Other:
- board outline added: 35 x 49 mm
