File: UccMicroDuino/UccMicroDuino.kicad_pcb (KiCad board)
At the start: 2 copper layers, 35 x 49 mm, 14 parts, among them J1 Conn_01x10_Socket, J2 USB_A, U1 ATtiny85-20S

Commit message: ruteo basico
Routing:
- net GND: track 0.00 -> 73.4 mm
- net Net-(J1-Pin_6): track 0.00 -> 31.8 mm
- net Net-(D5-K): track 0.04 -> 24.5 mm
- net Net-(D2-K): track 0.67 -> 12.8 mm
- net Net-(D1-A): track 0.71 -> 6.41 mm
- net +5V: track 0.00 -> 2.25 mm
