File: UccMicroDuino/UccMicroDuino.kicad_sch (KiCad schematic)
At the start: 8 parts, among them J2 Conn_01x10_Socket, J2 USB_A, U2 ATtiny85-20S

Commit message: Placa prueba didactica
Parts:
- added D4: LED, ledSmd:ledSMD, symbol Device:LED
- added D5: D_Zener, Diode_SMD:D_SOD-123, symbol Device:D_Zener
- added R2, R3, R4, R5: R, Resistor_SMD:R_0805_2012Metric_Pad1.20x1.40mm_HandSolder, symbol Device:R
Connections:
- net +5V: now also C1.1, D3.2 (A), J2.1 (Pin_1), U2.8 (VCC)
- net GND: now also C1.2, D1.2 (A), J2.2 (Pin_2), U2.4 (GND), D5.2 (A), R2.1, R3.1
- net at D3.1 (K): now also R3.2
- net at R1.2: now also J2.3 (D+), D5.1 (K), R5.2
- net at D1.1 (K): now also J2.2 (D-), R4.2
- net at U2.1 (~{RESET}/PB5): now also J2.10 (Pin_10)
- net at U2.2 (XTAL1/PB3): now also J2.7 (Pin_7), R4.1
- net at U2.3 (XTAL2/PB4): now also J2.8 (Pin_8)
- net at U2.5 (AREF/PB0): now also J2.4 (Pin_4)
- net at U2.6 (PB1): now also J2.5 (Pin_5), D4.2 (A)
- net at U2.7 (PB2): now also J2.6 (Pin_6), R5.1
- net at J2.1 (VBUS): now also D5.2 (A)
- new net: D4.1 (K), R2.2
- no-connect marks 0 -> 2
Other:
- moved on the sheet: D3, U2
