File: UccMicroDuino/UccMicroDuino.kicad_sch (KiCad schematic)
At the start: 14 parts, among them J2 Conn_01x10_Socket, J2 USB_A, U2 ATtiny85-20S

Commit message: 1011641-mi primer versionado con gitBash
Parts:
- renumbered D5 to D1, D1 to D2, J2 to J1, U2 to U1
Other:
- note added: "Circuito Principal"
- note removed: "Main Circuit"
- moved on the sheet: U1
